File: pcb/power-board/power-board.kicad_pcb (KiCad board)
At the start: 4 copper layers, 97 x 64.5 mm, 106 parts, among them J1 XT60 pack, J10 POWER button, J11 E-STOP button, J12 Control (ESP32), J2 Balance 3S, J3 LOGIC OUT, J4 Servo R leg, J5 Servo R upper, J6 Servo L leg, J7 Servo L upper, J8 Data from H5, J9 I2C (to P1), Q1 CSD17556Q5B, Q2 CSD17556Q5B, Q3 CSD17556Q5B, Q4 2N7002, Q5 MMBT3904, U1 BQ76922, U2 TPS48111-Q1

Commit message: Power board rev B: the board changes from the 2026-10-24 records
Schematic (generated from the rev A pipeline, ERC 0, netlist matches its spec):
- F-1: R38/R39 4.7k/1k and R41 4.7k from PACK+ to GND, so SHUTDOWN completes
  after KILL.
- F-2: D2 BAT54C -> Diodes BAV70 (silicon, same SOT-23 pinout; leakage at the
  1N4148W's limits the fix was simulated with) and R10 10k -> 100k.
- F-5: D10, a 15 V zener (MMSZ5245B) from Q3's gate to its source, and R43, a
  0 R gate placeholder at Q3 (layout review M1).
- F-7: C24-C27, 4 x 10 uF on PACK+ as two series pairs (one cracked part
  cannot short PACK+).
- F-9: R42 1k from J2.1 to BAT-.
- Audit F3: R29 10k, R30 549k. Audit F4: C28 1 nF across Q5.
- Value labels match the MPNs (C5-C8, C9-C11, C15, C18, C20, C22, C23);
  TI maker names; datasheet links (C15, C17, J1).
- J11 (E-STOP) is a JST ZH 4-pin, a family no other lead here uses (W1).
- J1, F1, F2 are do-not-populate (hand-soldered); TP1-TP8 off the BOM.

Layout (pipeline route b1; DRC 0 violations, 0 unconnected; every power pour
one piece):
- Q3's gate: R43 and D10 at the gate pad; SRV_G by B.Cu under Q3 to R28,
  about 10 mm instead of the 37 mm hairpin through the SERVO+ pour (M1).
- CSD17556Q5B paste per TI 7.3 (M2); C4 on REG18's F.Cu path, no vias (M3);
  R1's GND pour over its pad and 20 vias (M8); stray "J10" text gone (W1);
  legends 1.0 mm, references 0.8 x 0.15 mm (PCBWay's minimum, C3).
- 1 oz outer copper kept. fab/ regenerated by fab.sh (BOM without J1/F1/F2/TP).

Whole-board model: BAV70 and MMSZ5245B models, a 0 R resistor, rev A's
what-ifs that rev B now carries removed (62 sequences, 113 sweeps); the
behavioural models and schematic tests follow the new values.

Datasheets: Diodes BAV70, JST ZH.

Gates: make pytest - tests/ 380 passed, 16 skipped, 1 xfailed; pbsim 88
passed, 3 xfailed.

Co-Authored-By: Claude Opus 5.5 <noreply@anthropic.com>
Parts:
- added C24: 10u 35V, Capacitor_SMD:C_1206_3216Metric, F.Cu at (157.5, 70.0)
- added C25: 10u 35V, Capacitor_SMD:C_1206_3216Metric, F.Cu at (162.2, 70.0)
- added C26: 10u 35V, Capacitor_SMD:C_1206_3216Metric, F.Cu at (157.5, 73.0)
- added C27: 10u 35V, Capacitor_SMD:C_1206_3216Metric, F.Cu at (162.2, 73.0)
- added C28: 1n 50V, Capacitor_SMD:C_0603_1608Metric, F.Cu at (166.6, 86.8)
- added D10: 15V, Diode_SMD:D_SOD-123, F.Cu at (171.9, 77.7)
- added R41: 4.7k, Resistor_SMD:R_0603_1608Metric, F.Cu at (157.5, 75.4)
- added R42: 1k, Resistor_SMD:R_0603_1608Metric, F.Cu at (118.0, 93.0)
- added R43: 0, Resistor_SMD:R_0603_1608Metric, F.Cu at (167.6, 75.2)
- C10: value 100p -> 100p 50V
- C11, C18, C20: value 10n -> 10n 50V
- C15: value 1n -> 1n 50V
- C22: value 10u 25V -> 10u 35V
- C23, C9: value 100n -> 100n 50V
- C5, C6, C7, C8: value 100n 25V -> 100n 50V
- D2: value BAT54C -> BAV70
- J11: footprint Connector_JST:JST_PH_B4B-PH-K_1x04_P2.00mm_Vertical -> Connector_JST:JST_ZH_B4B-ZR_1x04_P1.50mm_Vertical
- R10: value 10k -> 100k
- R29: value 1k -> 10k
- R30: value 560k -> 549k
- R38: value 47k -> 4.7k
- R39: value 10k -> 1k
- moved C4 2.12 mm to (122.1, 106.6), turned to 180 degrees
Connections:
- Q3 pad 4: Net-(Q3-G) -> Net-(D10-K)
- R27 pad 2: Net-(Q3-G) -> Net-(U2-PD)
- R28 pad 1: Net-(Q3-G) -> Net-(U2-PD)
- U2 pad 14: Net-(Q3-G) -> Net-(U2-PD)
Routing:
- net Net-(Q3-G): track 37.5 -> 0.00 mm, vias 2 -> 0
- net Net-(U2-PD): track 0.00 -> 20.7 mm, vias 0 -> 2
- net PACK+: track 91.7 -> 83.3 mm, vias 15 -> 20
- net /SERVO_IMON: track 45.6 -> 53.1 mm
- net /RAIL_V: track 54.4 -> 61.0 mm
- net Net-(U1-REG18): track 8.21 -> 2.13 mm, vias 2 -> 0
- net Net-(D10-K): track 0.00 -> 4.77 mm
- net SERVO+: track 15.1 -> 19.0 mm, vias 109 -> 113
- net Net-(C16-Pad1): track 10.2 -> 14.0 mm
- net GND: track 32.8 -> 36.7 mm, vias 269 -> 287
- net Net-(J11-Pin_1): track 38.1 -> 35.3 mm, vias 2 -> 1
- net Net-(Q3-D): track 17.9 -> 15.2 mm
- net Net-(J2-Pin_1): track 7.89 -> 10.5 mm
- net Net-(C26-Pad2): track 0.00 -> 1.75 mm
- net Net-(C24-Pad2): track 0.00 -> 1.75 mm
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Other:
- board text added: "BIPED POWER rev B"
- board text removed: "BIPED POWER rev A"
- board text removed: "J10"
