File: pcb/power-board/power-board.kicad_sch (KiCad schematic)
At the start: 102 parts, among them J1 XT60 pack, J10 POWER button, J11 E-STOP button, J12 Control (ESP32), J2 Balance 3S, J3 LOGIC OUT, J4 Servo R leg, J5 Servo R upper, J6 Servo L leg, J7 Servo L upper, J8 Data from H5, J9 I2C (to P1), Q1 CSD17556Q5B, Q2 CSD17556Q5B, Q3 CSD17556Q5B, Q4 2N7002, Q5 MMBT3904, U1 BQ76922, U2 TPS48111-Q1

Commit message: Power board rev B: the board changes from the 2026-10-24 records
Schematic (generated from the rev A pipeline, ERC 0, netlist matches its spec):
- F-1: R38/R39 4.7k/1k and R41 4.7k from PACK+ to GND, so SHUTDOWN completes
  after KILL.
- F-2: D2 BAT54C -> Diodes BAV70 (silicon, same SOT-23 pinout; leakage at the
  1N4148W's limits the fix was simulated with) and R10 10k -> 100k.
- F-5: D10, a 15 V zener (MMSZ5245B) from Q3's gate to its source, and R43, a
  0 R gate placeholder at Q3 (layout review M1).
- F-7: C24-C27, 4 x 10 uF on PACK+ as two series pairs (one cracked part
  cannot short PACK+).
- F-9: R42 1k from J2.1 to BAT-.
- Audit F3: R29 10k, R30 549k. Audit F4: C28 1 nF across Q5.
- Value labels match the MPNs (C5-C8, C9-C11, C15, C18, C20, C22, C23);
  TI maker names; datasheet links (C15, C17, J1).
- J11 (E-STOP) is a JST ZH 4-pin, a family no other lead here uses (W1).
- J1, F1, F2 are do-not-populate (hand-soldered); TP1-TP8 off the BOM.

Layout (pipeline route b1; DRC 0 violations, 0 unconnected; every power pour
one piece):
- Q3's gate: R43 and D10 at the gate pad; SRV_G by B.Cu under Q3 to R28,
  about 10 mm instead of the 37 mm hairpin through the SERVO+ pour (M1).
- CSD17556Q5B paste per TI 7.3 (M2); C4 on REG18's F.Cu path, no vias (M3);
  R1's GND pour over its pad and 20 vias (M8); stray "J10" text gone (W1);
  legends 1.0 mm, references 0.8 x 0.15 mm (PCBWay's minimum, C3).
- 1 oz outer copper kept. fab/ regenerated by fab.sh (BOM without J1/F1/F2/TP).

Whole-board model: BAV70 and MMSZ5245B models, a 0 R resistor, rev A's
what-ifs that rev B now carries removed (62 sequences, 113 sweeps); the
behavioural models and schematic tests follow the new values.

Datasheets: Diodes BAV70, JST ZH.

Gates: make pytest - tests/ 380 passed, 16 skipped, 1 xfailed; pbsim 88
passed, 3 xfailed.

Co-Authored-By: Claude Opus 5.5 <noreply@anthropic.com>
Parts:
- added C24, C25, C26, C27: 10u 35V, Capacitor_SMD:C_1206_3216Metric, symbol Device:C
- added C28: 1n 50V, Capacitor_SMD:C_0603_1608Metric, symbol Device:C
- added D10: 15V, Diode_SMD:D_SOD-123, symbol Device:D_Zener
- added R41: 4.7k, Resistor_SMD:R_0603_1608Metric, symbol Device:R
- added R42: 1k, Resistor_SMD:R_0603_1608Metric, symbol Device:R
- added R43: 0, Resistor_SMD:R_0603_1608Metric, symbol Device:R
- C10: value 100p -> 100p 50V
- C11, C18, C20: value 10n -> 10n 50V
- C15: value 1n -> 1n 50V
- C22: value 10u 25V -> 10u 35V
- C23, C9: value 100n -> 100n 50V
- C5, C6, C7, C8: value 100n 25V -> 100n 50V
- D2: value BAT54C -> BAV70; symbol Diode:BAT54C -> Diode:BAV70; MPN Diotec BAT54C -> Diodes BAV70-7-F
- F1: MPN Keystone 3568 + Littelfuse 0297015.WXNV -> Keystone 3568; now not fitted
- F2: MPN Keystone 3568 + Littelfuse 0297003.WXNV -> Keystone 3568; now not fitted
- J1: now not fitted
- J11: footprint Connector_JST:JST_PH_B4B-PH-K_1x04_P2.00mm_Vertical -> Connector_JST:JST_ZH_B4B-ZR_1x04_P1.50mm_Vertical; MPN JST B4B-PH-K-S -> JST B4B-ZR(LF)(SN)
- Q1, Q2, Q3: MPN CSD17556Q5B -> TI CSD17556Q5B
- R10: value 10k -> 100k; MPN Yageo RC0603FR-0710KL -> Yageo RC0603FR-07100KL
- R29: value 1k -> 10k; MPN Yageo RC0603FR-071KL -> Yageo RC0603FR-0710KL
- R30: value 560k -> 549k; MPN Yageo RC0603FR-07560KL -> Yageo RC0603FR-07549KL
- R38: value 47k -> 4.7k; MPN Yageo RC0603FR-0747KL -> Yageo RC0603FR-074K7L
- R39: value 10k -> 1k; MPN Yageo RC0603FR-0710KL -> Yageo RC0603FR-071KL
- TP1, TP2, TP3, TP4, TP5, TP6, TP7, TP8: now left out of the parts list
- U1: MPN BQ76922RSNR -> TI BQ76922RSNR
- U2: MPN TPS48111LQDGXRQ1 -> TI TPS48111LQDGXRQ1
Connections:
- net BAT-: now also R42.2
- net GND: now also C25.2, C27.2, C28.2, R41.2
- net PACK+: now also C24.1, C26.1, R41.1
- net SERVO+: now also D10.2 (A)
- net at J2.1 (Pin_1), R3.1: now also R42.1
- net at R27.2, R28.1, U2.14 (PD): now also R43.2; no longer Q3.4 (G)
- net at Q5.1 (B), Q5.3 (C), U2.10 (DIODE): now also C28.1
- new net: C26.2, C27.1
- new net: C24.2, C25.1
- new net: D10.1 (K), Q3.4 (G), R43.1
Other:
- note added: "Rev B, 2026-10-29. Design: docs/design-v6/2026-10-06-power-circuit.md; checks: docs/design-v6/2026-10-07-power-board-verification.md and the 2026-10-24 records (full simulation, pin audit, layout review). J1, F1 and F2 are soldered by hand (DNP). Kelvin-route SRP/SRN (R7, R8) to the pads of R1, and CS+, CS-, ISCP to R24. Q5 against Q3, RT1 by Q1/Q2. Check against the real parts before ordering: X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"
- note removed: "Rev A, 2026-10-07. Design: docs/design-v6/2026-10-06-power-circuit.md; checks: docs/design-v6/2026-10-07-power-board-verification.md. Kelvin-route SRP/SRN (R7, R8) to the pads of R1, and CS+, CS-, ISCP to R24. Q5 against Q3, RT1 by Q1/Q2. Check against the real parts before ordering: XT60 polarity (J1), balance-lead order (J2), servo-header orientation (J4-J8 must mate like the General Driver's H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"
